File: 6.0/template/M5Stack_module_fdm/M5Stack_module_fdm.kicad_pcb (KiCad board)
At the start: 2 copper layers, 50 x 50 mm, 9 parts, among them U1 M-BUS

Commit message: template M5Stack
M-BUS connector  U1 to J1
Parts:
- removed U1: M-BUS, @bf:BF@M5Stack_MBUS
- added J1: M-BUS, @bf:BF@M5Stack_MBUS, F.Cu at (108.0, 127.0)
